File: Browse/nixie.kicad_pcb (KiCad board)
At the start: 4 copper layers, 189 x 55 mm, 70 parts, among them J1 Barrel_Jack, J2 Conn_01x02_Pin, Q1 2N3906, Q2 IRF644, SW1 RotaryEncoder_Switch, U1 4504, U2 MC34063AP, U3 HV5222PG-G, U4 LM7805_TO220, U5 HV5222PG-G, U6 ATmega328P-P, U7 DS3231MZ

Commit message: Deploying to gh-pages from @ pimborman/nixie-clock@de780db2857f2b30e7a47e9d26594c67cc7b3d3c 🚀
Parts:
- R2: value R -> 800k
- R3: value R -> 4.7k
- R4: value R -> 1
Changed lines of the file:
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@@
 		(at 108.12 85 90)
 		(descr "Potentiometer, vertical, Bourns 3386P, https://www.bourns.com/pdfs/3386.pdf")
-		(tags "Potentiometer vertical Bourns 3386P")
+		(tags "Potentiometer vertical Bourns 3306P")
 		(property "Reference" "RV1"
 			(at -4.8 -2.32 180)
@@
 			(layer "F.Fab")
 		)
+		(fp_text user "${REFERENCE}"
+			(at -4.95 -3.05 180)
+			(layer "F.Fab")
+			(effects
+				(font
+					(size 1 1)
+					(thickness 0.15)
+				)
+			)
+		)
 		(pad "1" thru_hole circle
 			(at 0 0 90)
@@
 			(pintype "passive")
 		)
-		(model "${KIPRJMOD}/packages3D/Potentiometer_Bourns_3386P_Vertical.wrl"
+		(model "${KIPRJMOD}/packages3D/3306P-1-103.step"
 			(offset
-				(xyz 0 0 0)
+				(xyz 1.25 2.5 0)
 			)
 			(scale
@@
 			)
 			(rotate
-				(xyz 0 0 0)
+				(xyz -90 0 90)
 			)
 		)
@@
 			)
 		)
-		(property "Value" "R"
+		(property "Value" "1"
 			(at 3.9 -0.08 90)
 			(layer "F.SilkS")
@@
 			)
 		)
-		(property "Value" "R"
+		(property "Value" "800k"
 			(at 3.92 0.08 90)
 			(layer "F.SilkS")
@@
 			)
 		)
-		(property "Value" "R"
+		(property "Value" "4.7k"
 			(at 3.81 0.08 90)
 			(layer "F.SilkS")
