File: Browse/nixie.kicad_sch (KiCad schematic)
At the start: 52 parts, among them J1 Barrel_Jack, J2 Conn_01x02_Pin, Q1 2N3906, Q2 IRF644, U1 4504, U2 MC34063AP, U3 HV5222PG-G, U4 LM7805_TO220, U5 HV5222PG-G

Commit message: Deploying to gh-pages from @ pimborman/nixie-clock@de780db2857f2b30e7a47e9d26594c67cc7b3d3c 🚀
Parts:
- R2: value R -> 800k
- R3: value R -> 4.7k
- R4: value R -> 1
Changed lines of the file:
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@@
     (stroke (width 0) (type default))
   )
-  (rectangle (start 12.7 14.478) (end 132.08 90.678)
+  (rectangle (start 12.7 14.478) (end 132.08 93.218)
     (stroke (width 0.2) (type dash))
     (fill (type none))
@@
       (effects (font (size 1.27 1.27)) (justify right))
     )
-    (property "Value" "R" (at 101.6 74.9299 0)
+    (property "Value" "4.7k" (at 101.6 74.9299 0)
       (effects (font (size 1.27 1.27)) (justify right))
     )
@@
       (effects (font (size 1.27 1.27)) (justify right))
     )
-    (property "Value" "R" (at 101.6 64.7699 0)
+    (property "Value" "800k" (at 101.6 64.7699 0)
       (effects (font (size 1.27 1.27)) (justify right))
     )
@@
       (effects (font (size 1.27 1.27)) (justify left))
     )
-    (property "Value" "R" (at 111.76 50.7999 0)
-      (effects (font (size 1.27 1.27)) (justify left))
-    )
+    (property "Value" "1" (at 111.76 50.7999 0)
+      (effects (font (size 1.27 1.27)) (justify left))
+    )
